File: Radxa_HAT_communications/hardware/HAT_communication_protocols/HAT_communication_protocols.kicad_pcb (KiCad board)
At the start: 2 copper layers, 68.1 x 58 mm, 74 parts, among them J1 Conn_01x02_Pin, J2 Can_terminals, J3 120Can-resistor, J4 PS-12V, J5 LoRa_DIO, J6 PoE, Q1 NMOS, U1 AMS1117-5.0, U2 MP2307, U3 74HC04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

Commit message: PCB V1.3 done
Parts:
- added -: Symbol_GNU-Logo_SilkscreenTop, Symbol:Symbol_GNU-Logo_SilkscreenTop, F.Cu at (145.2, 79.7)
- added Engineered by : LOGO, FourierEmbed2.preety:LOGOFOURIEREMBEDS, F.Cu at (158.3, 80.6)
- added REF**: ESD-Logo_6.6x6mm_SilkScreen, Symbol:ESD-Logo_6.6x6mm_SilkScreen, F.Cu at (179.3, 84.8)
- renumbered J4 to 12V-IN, J2 to CAN, RS485_interface1 to RS485, uart_RX1 to RX, RadxaGPIO1 to Radxa-IO, uart_TX1 to TX
Routing:
- net GND: vias 22 -> 63
- net (no net): vias 57 -> 0
Other:
- board text added: "Engineered by: Adrián Silva Palafox Felipe Adriel Trejo de Arcos"
