File: Radxa_HAT_communications/hardware/HAT_communication_protocols/HAT_communication_protocols.kicad_pcb (KiCad board)
At the start: 2 copper layers, 68.1 x 58 mm, 77 parts, among them J1 Conn_01x02_Pin, J3 120Can-resistor, J5 LoRa_DIO, J6 PoE, Q1 NMOS, U1 AMS1117-5.0, U2 MP2307, U3 74HC04, U4 MAX3485, U5 MCP2515-xSO, U6 TJA1051T-3, U7 LD1117V33, Y1 8MHz

Commit message: PCB V1.4 done
Parts:
- added TP1: TestPoint_Probe, TestPoint:TestPoint_Pad_D1.0mm, F.Cu at (150.5, 89.2)
- added TP2: TestPoint_Probe, TestPoint:TestPoint_Pad_D1.0mm, F.Cu at (177.3, 99.1)
- added TP3: TestPoint_Probe, TestPoint:TestPoint_Pad_D1.0mm, B.Cu at (127.6, 83.8)
- added TP4: TestPoint_Probe, TestPoint:TestPoint_Pad_D1.0mm, F.Cu at (131.6, 118.8)
- added TP5: TestPoint_Probe, TestPoint:TestPoint_Pad_D1.0mm, F.Cu at (142.2, 91.4)
- moved REF** 6.38 mm to (180.1, 91.1)
- renumbered C14 to C1, C5 to C10, C19 to C11, C18 to C12, C16 to C13, C1 to C14, C4 to C15, C7 to C16, C15 to C17, C3 to C18, C13 to C2, C11 to C3, C10 to C4, C9 to C5, C17 to C6, C12 to C7, C6 to C9, D4 to D1, D5 to D2, D6 to D3, D7 to D4, D3 to D5, D8 to D6, D2 to D7, D9 to D8, D1 to D9, F2 to F1, F3 to F2, F1 to F3, CAN to J2, J5 to J4, 12V-IN to J5, L2 to L1, R5 to R1, R12 to R11, R13 to R12, R14 to R13, R15 to R14, R16 to R15, R17 to R16, R1 to R17, R6 to R5, R11 to R6, U3 to U1, U5 to U2, U4 to U3, U6 to U4, U1 to U5, U7 to U6, U2 to U7
Connections:
- Radxa-IO pad 29: /GPIO07 -> /CAN_INT
- SX1 pad 6: /LoRa_RST -> /GPIO11
Routing:
- net /GPIO11: track 0.00 -> 17.8 mm
- net /CAN_INT: track 0.00 -> 17.7 mm
- net PS+5v: track 57.2 -> 59.1 mm
- net PS+6.2v: track 69.2 -> 70.0 mm

Commit message: PCB V1.5 done
Parts:
- removed the REF** at (180.1, 91.1)
- added REF**: OSHW-Logo_11.4x12mm_SilkScreen, Symbol:OSHW-Logo_11.4x12mm_SilkScreen, F.Cu at (157.2, 80.5)
- Engineered by : moved to B.Cu
- moved Engineered by  17.1 mm to (141.4, 83.4), turned to 180 degrees
- moved - 0.18 mm to (145.2, 79.5)
- renumbered J2 to CAN, J5 to Vin-12V
Other:
- board text added: "*Engineered by: Adrián Silva Palafox Felipe Adriel Trejo de Arcos *Full documentation on: GitHub: La-guajolota/Radxa-x4-devs"
- board text removed: "Engineered by: Adrián Silva Palafox Felipe Adriel Trejo de Arcos"

Commit message: Final Review - in production
Routing:
- net Net-(D2-A1): track 28.3 -> 25.8 mm
Other:
- board size 68.1 x 58 mm -> 66 x 58 mm
- board text added: "*Engineered by: Adrián Silva Palafox Felipe Adriel Trejo De Arcos *Full documentation on: GitHub: La-guajolota/Radxa-x4-devs"
- board text removed: "*Engineered by: Adrián Silva Palafox Felipe Adriel Trejo de Arcos *Full documentation on: GitHub: La-guajolota/Radxa-x4-devs"
