File: Radxa_HAT_communications/hardware/HAT_communication_protocols/HAT_communication_protocols.kicad_sch (KiCad schematic)
At the start: 79 parts, among them J1 Conn_01x02_Pin, J2 Can_terminals, J3 120Can-resistor, J4 LoRa_DIO, J5 PS-12V, J6 PoE, Q1 NMOS, U1 74HC04, U2 MCP2515-xSO, U3 MAX3485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

Commit message: Final Review - in production
Other:
- note added: "Mounting holes | pins-header | terminal-blocks"
- note removed: "Mounting holes | pins-header | termianl-blocks"
